Commit message: added gazebo simulator option for computers without NVIDIA GPU (unable to run IsaacSim)

File: src/amm_description/urdf/ridgeback_franka.urdf.xacro (robot description, xacro)
@@ -5,14 +5,18 @@
   Combines the Clearpath Ridgeback omnidirectional mobile base with the
   Franka FR3 7-DoF arm mounted on the top plate.
+  Arguments:
+    use_gazebo   (default false) — include Gazebo Harmonic plugins
+    sim_gazebo   (default false) — alias, same effect
   Dependencies (must be installed / cloned into your workspace):
     - ridgeback_description   (ros-jazzy-ridgeback-description or from source)
     - franka_description      (from franka_ros2, Jazzy branch)
-  The full robot model is already available as a native USD asset inside
-  Isaac Sim: Robots/Clearpath/Ridgeback/ridgeback_franka.usd
-  This URDF is used by ROS 2 tools (RViz2, MoveIt, TF tree) only.
   Usage:
     ros2 launch amm_description description.launch.py
+    xacro ridgeback_franka.urdf.xacro use_gazebo:=true
 -->
 <robot xmlns:xacro="http://www.ros.org/wiki/xacro" name="ridgeback_franka">
+  <!-- ── Arguments ─────────────────────────────────────────────────────────── -->
+  <xacro:arg name="use_gazebo"  default="false"/>
+  <xacro:arg name="sim_gazebo"  default="false"/>
   <!-- ── Ridgeback base ──────────────────────────────────────────────────────── -->
   <xacro:include filename="$(find ridgeback_description)/urdf/ridgeback.urdf.xacro"/>
@@ -20,10 +24,4 @@
   <xacro:include filename="$(find franka_description)/robots/fr3/fr3.urdf.xacro"/>
   <!-- ── Mount the arm on the Ridgeback top plate ───────────────────────────── -->
-  <!--
-    The Ridgeback top plate link is "mid_mount".
-    The arm is attached with a fixed joint so that the FR3 base aligns
-    with the centre of the Ridgeback chassis.
-    Adjust xyz/rpy to match the physical or simulated mounting position.
-  -->
   <joint name="ridgeback_to_fr3" type="fixed">
     <parent link="mid_mount"/>
@@ -32,5 +30,180 @@
   </joint>
   <!-- ── Franka Hand (parallel gripper) ────────────────────────────────────── -->
-  <!-- The Franka Hand is included as part of fr3.urdf.xacro above.            -->
-  <!-- End-effector TCP link: fr3_hand_tcp                                      -->
+  <!-- Included as part of fr3.urdf.xacro above.  TCP: fr3_hand_tcp            -->
+  <!-- ══════════════════════════════════════════════════════════════════════════
+       GAZEBO HARMONIC PLUGINS
+       Only included when use_gazebo:=true or sim_gazebo:=true.
+       ══════════════════════════════════════════════════════════════════════════ -->
+  <xacro:if value="$(eval '$(arg use_gazebo)' == 'true' or '$(arg sim_gazebo)' == 'true')">
+    <!-- ── gz_ros2_control — arm + gripper joints ──────────────────────────── -->
+    <gazebo>
+      <plugin filename="gz_ros2_control-system"
+              name="gz_ros2_control::GazeboSimROS2ControlPlugin">
+        <parameters>$(find amm_bringup)/config/manipulation.yaml</parameters>
+        <ros>
+          <namespace>/</namespace>
+        </ros>
+      </plugin>
+    </gazebo>
+    <!-- ── Mecanum drive controller — Ridgeback base ───────────────────────── -->
+    <!--
+      The mecanum_drive_controller plugin drives the four mecanum wheels by
+      reading /cmd_vel (geometry_msgs/Twist) and publishing /odom.
+      Wheel joint names must match ridgeback_description.
+    -->
+    <gazebo>
+      <plugin filename="gz-sim-mecanum-drive-system"
+              name="gz::sim::systems::MecanumDrive">
+        <front_left_joint>front_left_wheel</front_left_joint>
+        <front_right_joint>front_right_wheel</front_right_joint>
+        <rear_left_joint>rear_left_wheel</rear_left_joint>
+        <rear_right_joint>rear_right_wheel</rear_right_wheel>
+        <wheel_separation>0.476</wheel_separation>
+        <wheelbase>0.476</wheelbase>
+        <wheel_radius>0.0875</wheel_radius>
+        <min_acceleration>-5</min_acceleration>
+        <max_acceleration>5</max_acceleration>
+        <topic>cmd_vel</topic>
+        <odom_topic>odom</odom_topic>
+        <frame_id>odom</frame_id>
+        <child_frame_id>base_link</child_frame_id>
+        <odom_publish_frequency>50</odom_publish_frequency>
+      </plugin>
+    </gazebo>
+    <!-- ── 2D LiDAR ─────────────────────────────────────────────────────────── -->
+    <!--
+      Mounted on the Ridgeback front; publishes sensor_msgs/LaserScan.
+      Bridged to /scan via ros_gz_bridge.
+    -->
+    <link name="lidar_link">
+      <visual>
+        <geometry><cylinder radius="0.04" length="0.05"/></geometry>
+        <material><ambient>0.2 0.2 0.2 1</ambient></material>
+      </visual>
+      <collision>
+        <geometry><cylinder radius="0.04" length="0.05"/></geometry>
+      </collision>
+      <inertial>
+        <mass>0.1</mass>
+        <inertia><ixx>0.0001</ixx><ixy>0</ixy><ixz>0</ixz>
+                 <iyy>0.0001</iyy><iyz>0</iyz><izz>0.0001</izz></inertia>
+      </inertial>
+    </link>
+    <joint name="lidar_joint" type="fixed">
+      <parent link="base_link"/>
+      <child  link="lidar_link"/>
+      <origin xyz="0.3 0.0 0.3" rpy="0 0 0"/>
+    </joint>
+    <gazebo reference="lidar_link">
+      <sensor name="lidar" type="gpu_lidar">
+        <update_rate>15</update_rate>
+        <topic>lidar/scan</topic>
+        <gz_frame_id>lidar_link</gz_frame_id>
+        <ray>
+          <scan>
+            <horizontal>
+              <samples>720</samples>
+              <resolution>1</resolution>
+              <min_angle>-3.14159</min_angle>
+              <max_angle>3.14159</max_angle>
+            </horizontal>
+          </scan>
+          <range>
+            <min>0.1</min>
+            <max>30.0</max>
+            <resolution>0.01</resolution>
+          </range>
+          <noise><type>gaussian</type><mean>0.0</mean><stddev>0.005</stddev></noise>
+        </ray>
+        <always_on>true</always_on>
+        <visualize>false</visualize>
+      </sensor>
+    </gazebo>
+    <!-- ── RGB-D camera (wrist-mounted) ──────────────────────────────────────── -->
+    <!--
+      Mounted on the arm's end-effector link for manipulation perception.
+      Publishes image + depth + point cloud.
+      Bridged via ros_gz_bridge.
+    -->
+    <link name="camera_link">
+      <visual>
+        <geometry><box size="0.04 0.10 0.04"/></geometry>
+        <material><ambient>0.1 0.1 0.1 1</ambient></material>
+      </visual>
+      <collision>
+        <geometry><box size="0.04 0.10 0.04"/></geometry>
+      </collision>
+      <inertial>
+        <mass>0.1</mass>
+        <inertia><ixx>0.0001</ixx><ixy>0</ixy><ixz>0</ixz>
+                 <iyy>0.0001</iyy><iyz>0</iyz><izz>0.0001</izz></inertia>
+      </inertial>
+    </link>
+    <joint name="camera_joint" type="fixed">
+      <parent link="fr3_hand"/>
+      <child  link="camera_link"/>
+      <origin xyz="0.0 0.0 0.10" rpy="0 0.3 0"/>
+    </joint>
+    <link name="camera_optical_frame"/>
+    <joint name="camera_optical_joint" type="fixed">
+      <parent link="camera_link"/>
+      <child  link="camera_optical_frame"/>
+      <origin xyz="0 0 0" rpy="-1.5708 0 -1.5708"/>
+    </joint>
+    <gazebo reference="camera_link">
+      <sensor name="rgbd_camera" type="rgbd_camera">
+        <update_rate>30</update_rate>
+        <topic>camera</topic>
+        <gz_frame_id>camera_optical_frame</gz_frame_id>
+        <camera>
+          <horizontal_fov>1.047</horizontal_fov>
+          <image>
+            <width>640</width>
+            <height>480</height>
+            <format>RGB_INT8</format>
+          </image>
+          <clip><near>0.1</near><far>10.0</far></clip>
+          <depth_camera>
+            <clip><near>0.1</near><far>10.0</far></clip>
+          </depth_camera>
+          <noise><type>gaussian</type><mean>0</mean><stddev>0.007</stddev></noise>
+        </camera>
+        <always_on>true</always_on>
+        <visualize>false</visualize>
+      </sensor>
+    </gazebo>
+    <!-- ── IMU ────────────────────────────────────────────────────────────────── -->
+    <link name="imu_link">
+      <inertial>
+        <mass>0.01</mass>
+        <inertia><ixx>0.00001</ixx><ixy>0</ixy><ixz>0</ixz>
+                 <iyy>0.00001</iyy><iyz>0</iyz><izz>0.00001</izz></inertia>
+      </inertial>
+    </link>
+    <joint name="imu_joint" type="fixed">
+      <parent link="base_link"/>
+      <child  link="imu_link"/>
+      <origin xyz="0 0 0.1" rpy="0 0 0"/>
+    </joint>
+    <gazebo reference="imu_link">
+      <sensor name="imu_sensor" type="imu">
+        <update_rate>200</update_rate>
+        <topic>imu/data</topic>
+        <gz_frame_id>imu_link</gz_frame_id>
+        <always_on>true</always_on>
+        <imu>
+          <angular_velocity>
+            <x><noise type="gaussian"><mean>0</mean><stddev>0.0004</stddev></noise></x>
+            <y><noise type="gaussian"><mean>0</mean><stddev>0.0004</stddev></noise></y>
+            <z><noise type="gaussian"><mean>0</mean><stddev>0.0004</stddev></noise></z>
+          </angular_velocity>
+          <linear_acceleration>
+            <x><noise type="gaussian"><mean>0</mean><stddev>0.017</stddev></noise></x>
+            <y><noise type="gaussian"><mean>0</mean><stddev>0.017</stddev></noise></y>
+            <z><noise type="gaussian"><mean>0</mean><stddev>0.017</stddev></noise></z>
+          </linear_acceleration>
+        </imu>
+      </sensor>
+    </gazebo>
+  </xacro:if>
 </robot>

Commit message: changed room layout, fixed robot description again

File: src/amm_description/urdf/ridgeback_franka.urdf.xacro (robot description, xacro)
@@ -17,6 +17,5 @@
 <robot xmlns:xacro="http://www.ros.org/wiki/xacro" name="ridgeback_franka">
   <!-- ── Arguments ─────────────────────────────────────────────────────────── -->
-  <xacro:arg name="use_gazebo"  default="false"/>
-  <xacro:arg name="sim_gazebo"  default="false"/>
+  <xacro:arg name="use_gazebo" default="false"/>
   <!-- ── Ridgeback base ──────────────────────────────────────────────────────── -->
   <xacro:include filename="$(find ridgeback_description)/urdf/ridgeback.urdf.xacro"/>
@@ -24,7 +23,11 @@
   <xacro:include filename="$(find franka_description)/robots/fr3/fr3.urdf.xacro"/>
   <!-- ── Mount the arm on the Ridgeback top plate ───────────────────────────── -->
+  <!-- Connect the FR3's root link ("base") to the Ridgeback top plate.
+       fr3.urdf.xacro creates a "base" link and connects fr3_link0 to it;
+       we must parent "base" here rather than fr3_link0, otherwise "base"
+       remains a disconnected second root and the URDF parser rejects the model. -->
   <joint name="ridgeback_to_fr3" type="fixed">
     <parent link="mid_mount"/>
-    <child  link="fr3_link0"/>
+    <child  link="base"/>
     <origin xyz="0.0 0.0 0.05" rpy="0 0 0"/>
   </joint>
@@ -35,5 +38,5 @@
        Only included when use_gazebo:=true or sim_gazebo:=true.
        ══════════════════════════════════════════════════════════════════════════ -->
-  <xacro:if value="$(eval '$(arg use_gazebo)' == 'true' or '$(arg sim_gazebo)' == 'true')">
+  <xacro:if value="$(arg use_gazebo)">
     <!-- ── gz_ros2_control — arm + gripper joints ──────────────────────────── -->
     <gazebo>
@@ -58,5 +61,5 @@
         <front_right_joint>front_right_wheel</front_right_joint>
         <rear_left_joint>rear_left_wheel</rear_left_joint>
-        <rear_right_joint>rear_right_wheel</rear_right_wheel>
+        <rear_right_joint>rear_right_wheel</rear_right_joint>
         <wheel_separation>0.476</wheel_separation>
         <wheelbase>0.476</wheelbase>
@@ -79,5 +82,5 @@
       <visual>
         <geometry><cylinder radius="0.04" length="0.05"/></geometry>
-        <material><ambient>0.2 0.2 0.2 1</ambient></material>
+        <material name="lidar_dark"><color rgba="0.2 0.2 0.2 1"/></material>
       </visual>
       <collision>
@@ -85,7 +88,6 @@
       </collision>
       <inertial>
-        <mass>0.1</mass>
-        <inertia><ixx>0.0001</ixx><ixy>0</ixy><ixz>0</ixz>
-                 <iyy>0.0001</iyy><iyz>0</iyz><izz>0.0001</izz></inertia>
+        <mass value="0.1"/>
+        <inertia ixx="0.0001" ixy="0" ixz="0" iyy="0.0001" iyz="0" izz="0.0001"/>
       </inertial>
     </link>
@@ -129,5 +131,5 @@
       <visual>
         <geometry><box size="0.04 0.10 0.04"/></geometry>
-        <material><ambient>0.1 0.1 0.1 1</ambient></material>
+        <material name="camera_dark"><color rgba="0.1 0.1 0.1 1"/></material>
       </visual>
       <collision>
@@ -135,7 +137,6 @@
       </collision>
       <inertial>
-        <mass>0.1</mass>
-        <inertia><ixx>0.0001</ixx><ixy>0</ixy><ixz>0</ixz>
-                 <iyy>0.0001</iyy><iyz>0</iyz><izz>0.0001</izz></inertia>
+        <mass value="0.1"/>
+        <inertia ixx="0.0001" ixy="0" ixz="0" iyy="0.0001" iyz="0" izz="0.0001"/>
       </inertial>
     </link>
@@ -176,7 +177,6 @@
     <link name="imu_link">
       <inertial>
-        <mass>0.01</mass>
-        <inertia><ixx>0.00001</ixx><ixy>0</ixy><ixz>0</ixz>
-                 <iyy>0.00001</iyy><iyz>0</iyz><izz>0.00001</izz></inertia>
+        <mass value="0.01"/>
+        <inertia ixx="0.00001" ixy="0" ixz="0" iyy="0.00001" iyz="0" izz="0.00001"/>
       </inertial>
     </link>
