Commit message: Refactor navigation and control parameters for improved robot functionality
- Updated planner server plugin syntax in nav2_params.yaml
- Added smoother_server and velocity_smoother configurations
- Introduced behavior_server and waypoint_follower parameters
- Enhanced docking_server and collision_monitor settings
- Modified joint naming convention in ridgeback.urdf.xacro
- Integrated ros2_control hardware interface for FR3 arm in ridgeback_franka.urdf.xacro
- Established controller spawners in gazebo_sim.launch.py
- Created controllers.yaml for managing joint state and trajectory controllers

File: src/amm_description/robots/common/franka_arm.ros2_control.xacro (robot description, xacro)
@@ -95,5 +95,8 @@
       <gazebo>
         <plugin filename="gz_ros2_control-system" name="gz_ros2_control::GazeboSimROS2ControlPlugin">
-          <parameters>$(find franka_gazebo_bringup)/config/franka_gazebo_controllers.yaml</parameters>
+          <parameters>$(find amm_bringup)/config/controllers.yaml</parameters>
+          <!-- Note: this block is only reached if ros2_control:=true is passed
+               directly to fr3.urdf.xacro, which is NOT done in the AMM bringup.
+               The AMM bringup uses the ros2_control block in ridgeback_franka.urdf.xacro. -->
         </plugin>
       </gazebo>

File: src/amm_description/urdf/ridgeback.urdf.xacro (robot description, xacro)
@@ -117,5 +117,5 @@
       </collision>
     </link>
-    <joint name="${name}" type="continuous">
+    <joint name="${name}_joint" type="continuous">
       <parent link="base_link"/>
       <child  link="${name}"/>

File: src/amm_description/urdf/ridgeback_franka.urdf.xacro (robot description, xacro)
@@ -36,9 +36,84 @@
        ══════════════════════════════════════════════════════════════════════════ -->
   <xacro:if value="$(arg use_gazebo)">
-    <!-- ── gz_ros2_control — arm + gripper joints ──────────────────────────── -->
+    <!-- ── ros2_control hardware interface — FR3 arm + gripper ──────────────── -->
+    <!--
+      We define this block directly here rather than delegating to fr3.urdf.xacro's
+      ros2_control arg, because passing gazebo:=true to fr3.urdf.xacro suppresses
+      the 'base' link creation (intended for standalone Gazebo spawning only), which
+      would break the ridgeback_to_fr3 joint that attaches to 'base'.
+    -->
+    <ros2_control name="FrankaHardwareInterface" type="system">
+      <hardware>
+        <plugin>gz_ros2_control/GazeboSimSystem</plugin>
+      </hardware>
+      <joint name="fr3_joint1">
+        <command_interface name="position"/>
+        <command_interface name="velocity"/>
+        <state_interface name="position"><param name="initial_value">0.0</param></state_interface>
+        <state_interface name="velocity"/>
+        <state_interface name="effort"/>
+      </joint>
+      <joint name="fr3_joint2">
+        <command_interface name="position"/>
+        <command_interface name="velocity"/>
+        <state_interface name="position"><param name="initial_value">${-pi/4}</param></state_interface>
+        <state_interface name="velocity"/>
+        <state_interface name="effort"/>
+      </joint>
+      <joint name="fr3_joint3">
+        <command_interface name="position"/>
+        <command_interface name="velocity"/>
+        <state_interface name="position"><param name="initial_value">0.0</param></state_interface>
+        <state_interface name="velocity"/>
+        <state_interface name="effort"/>
+      </joint>
+      <joint name="fr3_joint4">
+        <command_interface name="position"/>
+        <command_interface name="velocity"/>
+        <state_interface name="position"><param name="initial_value">${-3*pi/4}</param></state_interface>
+        <state_interface name="velocity"/>
+        <state_interface name="effort"/>
+      </joint>
+      <joint name="fr3_joint5">
+        <command_interface name="position"/>
+        <command_interface name="velocity"/>
+        <state_interface name="position"><param name="initial_value">0.0</param></state_interface>
+        <state_interface name="velocity"/>
+        <state_interface name="effort"/>
+      </joint>
+      <joint name="fr3_joint6">
+        <command_interface name="position"/>
+        <command_interface name="velocity"/>
+        <state_interface name="position"><param name="initial_value">${pi/2}</param></state_interface>
+        <state_interface name="velocity"/>
+        <state_interface name="effort"/>
+      </joint>
+      <joint name="fr3_joint7">
+        <command_interface name="position"/>
+        <command_interface name="velocity"/>
+        <state_interface name="position"><param name="initial_value">${pi/4}</param></state_interface>
+        <state_interface name="velocity"/>
+        <state_interface name="effort"/>
+      </joint>
+      <joint name="fr3_finger_joint1">
+        <command_interface name="position"/>
+        <state_interface name="position"><param name="initial_value">0.0</param></state_interface>
+        <state_interface name="velocity"/>
+        <state_interface name="effort"/>
+      </joint>
+      <!-- fr3_finger_joint2 is a mimic of finger_joint1 — no command interfaces allowed -->
+      <joint name="fr3_finger_joint2">
+        <param name="mimic">fr3_finger_joint1</param>
+        <param name="mechanically_reduced">1</param>
+        <state_interface name="position"/>
+        <state_interface name="velocity"/>
+        <state_interface name="effort"/>
+      </joint>
+    </ros2_control>
+    <!-- gz_ros2_control plugin — reads the <ros2_control> block above ─────── -->
     <gazebo>
       <plugin filename="gz_ros2_control-system"
               name="gz_ros2_control::GazeboSimROS2ControlPlugin">
-        <parameters>$(find amm_bringup)/config/manipulation.yaml</parameters>
+        <parameters>$(find amm_bringup)/config/controllers.yaml</parameters>
         <ros>
           <namespace>/</namespace>
@@ -55,8 +130,8 @@
       <plugin filename="gz-sim-mecanum-drive-system"
               name="gz::sim::systems::MecanumDrive">
-        <front_left_joint>front_left_wheel</front_left_joint>
-        <front_right_joint>front_right_wheel</front_right_joint>
-        <rear_left_joint>rear_left_wheel</rear_left_joint>
-        <rear_right_joint>rear_right_wheel</rear_right_joint>
+        <front_left_joint>front_left_wheel_joint</front_left_joint>
+        <front_right_joint>front_right_wheel_joint</front_right_joint>
+        <rear_left_joint>rear_left_wheel_joint</rear_left_joint>
+        <rear_right_joint>rear_right_wheel_joint</rear_right_joint>
         <wheel_separation>0.476</wheel_separation>
         <wheelbase>0.476</wheelbase>
