Commit message: Update controller parameters and add inertial properties for Franka hand

File: src/amm_description/end_effectors/common/franka_hand.xacro (robot description, xacro)
@@ -126,5 +126,4 @@
       <axis xyz="0 1 0" />
       <limit effort="100" lower="0.0" upper="0.04" velocity="0.2" />
-      <mimic joint="${ee_prefix}finger_joint1" />
       <dynamics damping="0.3" />
     </joint>

File: src/amm_description/urdf/ridgeback_franka.urdf.xacro (robot description, xacro)
@@ -27,5 +27,5 @@
     <parent link="mid_mount"/>
     <child  link="base"/>
-    <origin xyz="0.0 0.0 0.05" rpy="0 0 0"/>
+    <origin xyz="0.0 0.0 0.0" rpy="0 0 0"/>
   </joint>
   <!-- ── Franka Hand (parallel gripper) ────────────────────────────────────── -->
@@ -102,9 +102,8 @@
         <state_interface name="effort"/>
       </joint>
-      <!-- fr3_finger_joint2 is a mimic of finger_joint1 — no command interfaces allowed -->
+      <!-- fr3_finger_joint2 mirrors finger_joint1 — commanded in sync by the gripper controller -->
       <joint name="fr3_finger_joint2">
-        <param name="mimic">fr3_finger_joint1</param>
-        <param name="mechanically_reduced">1</param>
-        <state_interface name="position"/>
+        <command_interface name="position"/>
+        <state_interface name="position"><param name="initial_value">0.0</param></state_interface>
         <state_interface name="velocity"/>
         <state_interface name="effort"/>
@@ -141,4 +140,5 @@
         <topic>cmd_vel</topic>
         <odom_topic>odom</odom_topic>
+        <tf_topic>/tf</tf_topic>
         <frame_id>odom</frame_id>
         <child_frame_id>base_link</child_frame_id>
